File: Projekt2_ArduinoTestBoard/MultiBoard.brd (EAGLE design)
At the start: 158.4 x 80 mm, 1 part

Commit message: max485
Parts:
- added C_MAX485_1, C_MAX485_2: (no value), rcl:C0805
- added D1: CGRM4007-G, diode:SOD-123_MINI-SMA
- added MAX485: MAX485CSA, andereBauteile:SO08
- added R5, R6: (no value), rcl:M0805
- added R_MAX1, R_MAX2, R_MAX3, R_MAX4, R_MAX485, R_MAX485_1, R_MAX485_2, R_MAX485_3: 10K, rcl:R0402
- added SV1: (no value), con-lsta:FE05-1
Connections:
- new net +5V: C_MAX485_1.1, C_MAX485_2.1, MAX485.8, R_MAX1.2, R_MAX2.2, R_MAX485.2, R_MAX485_1.2, R_MAX485_2.2, R_MAX485_3.2
- new net N$1: MAX485.1, R_MAX485_3.1
- new net N$2: MAX485.2, R_MAX485_2.1
- new net N$3: MAX485.3, R_MAX485_1.1
- new net N$4: MAX485.4, R_MAX485.1
- new net N$5: MAX485.7, R_MAX2.1, R_MAX4.2
- new net N$6: D1.A, R_MAX1.1
- new net N$7: MAX485.6, R_MAX3.2, R_MAX4.1
- net GND: now also C_MAX485_1.2, C_MAX485_2.2, D1.C, MAX485.5, R_MAX3.1
