File: Projekt2_ArduinoTestBoard/MultiBoard.brd (EAGLE design)
At the start: 158.4 x 62.2 mm, 29 parts, among them IC1 7805DT, X1 POWERSUPPLY_DC21MMX, Y1 16MHz

Commit message: Update PCB
Parts:
- added 485B: (no value), con-wago-508:W237-132
- added C1, C2: 22p, SmartPrj:C0603-ROUND
- added IC2: TJA1050, Marco:DIL08
- added JP_MAX485: (no value), jumper:JP4Q
- added U$2: MCP2515, mcp2515:TSSOP20
- added Y2: 8MHz, SmartPrj:QS
- moved PC2 303.1 mm to (16.5, 71.1), turned to 180 degrees
- moved PC1 297.3 mm to (29.2, 71.1)
- moved JP2 263.0 mm to (111.8, 25.4), turned to 90 degrees
- moved C_MAX485_2 242.1 mm to (49.5, 62.9), turned to 90 degrees
- moved RESET 240.3 mm to (7.62, 38.1)
- moved C_MAX485_1 230.0 mm to (50.8, 62.9), turned to 90 degrees
- moved ARDUINO 224.0 mm to (6.35, 30.5)
- moved R_MAX4 222.3 mm to (54.6, 64.8), turned to 180 degrees
- moved R_MAX3 217.1 mm to (56.5, 63.9), turned to 90 degrees
- moved R_MAX2 211.1 mm to (52.7, 63.9), turned to 270 degrees
- moved C9 194.3 mm to (35.6, 2.54)
- moved C11 192.7 mm to (11.4, 3.81), turned to 180 degrees
- moved R_MAX1 190.1 mm to (46.5, 52.1)
- moved Y1 185.7 mm to (20.3, 3.81)
- moved R1 183.4 mm to (29.2, 3.81)
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Connections:
- removed net IO0: ZU4.2
- removed net IO1: ZU4.3
- new net N$23: JP2.15, U$1.D12
- new net N$25: JP2.14, U$1.D11
- new net N$26: JP2.13, U$1.D10
- new net N$27: JP2.12, U$1.D9
- new net N$28: JP2.11, U$1.D8
- new net N$29: JP2.10, U$1.D7
- new net N$30: JP2.9, U$1.D6
- new net N$31: JP2.8, U$1.D5
- new net N$32: JP2.7, U$1.D4
- new net N$33: C1.1, U$2.8, Y2.1
- new net N$34: JP2.5, U$1.D2
- new net N$36: JP2.3, U$1.RST1
- new net N$37: C2.1, U$2.9, Y2.2
- new net RESET: ARDUINO.1, JP1.13, RESET.3, RESET.4, U$1.RST, ZU4.1
- new net RX: JP2.2, JP_MAX485.8, U$1.RX1, ZU4.2
- new net TX: JP2.1, JP_MAX485.2, U$1.TX0, ZU4.3
- net +5V: now also IC2.3
- net GND: now also C1.2, C2.2, IC2.2, JP2.4, U$1.GND1
- net IO3: now also JP2.6, JP_MAX485.4, JP_MAX485.6, U$1.D3
- net N$1: now also JP_MAX485.7
- net N$10: now also IC2.1, U$2.1; no longer ARDUINO.1, RESET.3, RESET.4, ZU4.1
- net N$2: now also JP_MAX485.5
- net N$22: now also IC2.4, U$2.2; no longer JP1.13, U$1.RST
- net N$3: now also JP_MAX485.3
- net N$4: now also JP_MAX485.1
- net N$5: now also 485B.2
- net N$7: now also 485B.1
Routing:
- net GND: track 0.00 -> 12.0 mm
- net N$5: track 0.00 -> 11.5 mm
- net N$7: track 0.00 -> 11.4 mm
- net N$4: track 0.00 -> 10.7 mm
- net N$1: track 0.00 -> 10.7 mm
- net N$3: track 0.00 -> 10.2 mm
- net N$2: track 0.00 -> 10.2 mm
- net TX: track 0.00 -> 5.08 mm
- net RX: track 0.00 -> 5.08 mm
- net RESET: track 0.00 -> 5.08 mm
- net N$9: track 0.00 -> 5.08 mm
- net N$36: track 0.00 -> 5.08 mm
- net N$34: track 0.00 -> 5.08 mm
- net N$32: track 0.00 -> 5.08 mm
- net N$31: track 0.00 -> 5.08 mm
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Other:
- board size 158.4 x 62.2 mm -> 116.5 x 76.2 mm
- board text added: "2x 1 µ"
- board text added: "4x10K"
- board text added: "MAX485"
