File: Projekt2_ArduinoTestBoard/MultiBoard.sch (EAGLE design)
At the start: 1 part

Commit message: max485
Parts:
- added C_MAX485_1, C_MAX485_2: (no value), rcl:C-EUC0805
- added D1: CGRM4007-G, diode:CGRM4007-G
- added MAX485: MAX485CSA, andereBauteile:MAX485CSA
- added R5, R6: (no value), rcl:R-EU_M0805
- added R_MAX1, R_MAX2, R_MAX3, R_MAX4, R_MAX485, R_MAX485_1, R_MAX485_2, R_MAX485_3: 10K, rcl:R-EU_R0402
- added SV1: (no value), con-lsta:FE05-1
Connections:
- new net +5V: C_MAX485_1.1, C_MAX485_2.1, MAX485G.VCC, R_MAX1.2, R_MAX2.2, R_MAX485.2, R_MAX485_1.2, R_MAX485_2.2, R_MAX485_3.2
- new net GND: C_MAX485_1.2, C_MAX485_2.2, D1.C, MAX485G.GND, R_MAX3.1
- new net N$1: MAX485G$1.RO, R_MAX485_3.1
- new net N$2: MAX485G$1.RE/, R_MAX485_2.1
- new net N$3: MAX485G$1.DE, R_MAX485_1.1
- new net N$4: MAX485G$1.DI, R_MAX485.1
- new net N$5: MAX485G$1.B, R_MAX2.1, R_MAX4.2
- new net N$6: D1.A, R_MAX1.1
- new net N$7: MAX485G$1.A, R_MAX3.2, R_MAX4.1
