File: Projekt2_ArduinoTestBoard/MultiBoard.sch (EAGLE design)
At the start: 29 parts, among them IC1 7805DT, X1 POWERSUPPLY_DC21MMX, Y1 16MHz

Commit message: Update PCB
Parts:
- added 485B: (no value), con-wago-508:W237-02P
- added C1, C2: 22p, SmartPrj:C-EU0603-RND
- added IC2: TJA1050, Marco:TJA1050
- added JP_MAX485: (no value), jumper:JP4Q
- added U$2: MCP2515, mcp2515:MCP2515
- added Y2: 8MHz, SmartPrj:XTAL/S
Connections:
- removed net IO0: ZU4.(RXD)PD0
- removed net IO1: ZU4.(TXD)PD1
- new net N$23: JP2.15, U$1.D12
- new net N$25: JP2.14, U$1.D11
- new net N$26: JP2.13, U$1.D10
- new net N$27: JP2.12, U$1.D9
- new net N$28: JP2.11, U$1.D8
- new net N$29: JP2.10, U$1.D7
- new net N$30: JP2.9, U$1.D6
- new net N$31: JP2.8, U$1.D5
- new net N$32: JP2.7, U$1.D4
- new net N$33: C1.1, U$2.OSC2, Y2.1
- new net N$34: JP2.5, U$1.D2
- new net N$36: JP2.3, U$1.RST1
- new net N$37: C2.1, U$2.OSC1, Y2.2
- new net RESET: ARDUINO.1, JP1.13, RESET.3, RESET.4, U$1.RST, ZU4.RESET
- new net RX: JP2.2, JP_MAX485.8, U$1.RX1, ZU4.(RXD)PD0
- new net TX: JP2.1, JP_MAX485.2, U$1.TX0, ZU4.(TXD)PD1
- net +5V: now also IC2.VCC
- net GND: now also C1.2, C2.2, IC2.GND, JP2.4, U$1.GND2
- net IO3: now also JP2.6, JP_MAX485.4, JP_MAX485.6, U$1.D3
- net N$1: now also JP_MAX485.7
- net N$10: now also IC2.TXD, U$2.TXCAN; no longer ARDUINO.1, RESET.3, RESET.4, ZU4.RESET
- net N$2: now also JP_MAX485.5
- net N$22: now also IC2.RXD, U$2.RXCAN; no longer JP1.13, U$1.RST
- net N$3: now also JP_MAX485.3
- net N$4: now also JP_MAX485.1
- net N$5: now also 485B-2.KL
- net N$7: now also 485B-1.KL
Other:
- note added: "Power Supply"
- moved on the sheet: MAX485G$1
