File: Projekt2_ArduinoTestBoard/1_PCB/MultiBoard.brd (EAGLE design)
At the start: 116.5 x 76.2 mm, 39 parts, among them IC1 7805DT, IC2 TJA1050, X1 POWERSUPPLY_DC21MMX, Y1 16MHz, Y2 8MHz

Commit message: PCB Update
Parts:
- moved R_MAX5 201.2 mm to (105.9, 51.4)
- moved C4 200.6 mm to (105.8, 55.9)
- moved C3 193.7 mm to (105.9, 53.1)
- moved C2 171.2 mm to (82.5, 49.5), flipped to the bottom
- moved C1 170.2 mm to (82.5, 54.6), flipped to the bottom
- moved IC2 168.0 mm to (99.1, 59.7)
- moved Y2 163.9 mm to (88.9, 52.1), turned to 270 degrees
- moved U$2 155.8 mm to (99.1, 49.5)
- moved PC2 8.98 mm to (15.2, 62.2)
- moved PC1 7.73 mm to (30.5, 63.5)
- moved IC1 5.08 mm to (22.9, 68.6), turned to 0 degrees
Connections:
- removed net N$24: JP1.15, U$1.RAW
- net PWRIN: now also JP1.15, U$1.RAW
Routing:
- net IO12: track 5.08 -> 25.3 mm
- net SPIMOSI: track 5.08 -> 23.2 mm, vias 0 -> 1
- net N$33: track 0.00 -> 16.7 mm
- net SPISCK: track 5.08 -> 21.8 mm
- net IO13: track 5.08 -> 21.1 mm
- net N$37: track 0.00 -> 13.4 mm
- net +5V: track 5.08 -> 18.3 mm
- net N$22: track 0.00 -> 9.29 mm
- net SPIMISO: track 5.08 -> 14.3 mm
- net PWRIN: track 0.00 -> 5.08 mm
- net N$24: track 5.08 -> 0.00 mm
- net N$10: track 0.00 -> 3.92 mm
- net N$23: track 0.00 -> 3.09 mm
