File: Projekt2_ArduinoTestBoard/1_PCB/V2/MultiboardV2.sch (EAGLE design)
At the start: 67 parts, among them IC1 MC33269ST-5.0T3, IC2 MC33269D-5.0, Q1 16MHz, Q2 16MHz, T1 FDN304V, U1 LM358D, U2 LP2985-33DBVR, U3 ATMEGA8U2-MU, X1 DC21MMX, Y1 16MHz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

Commit message: Added SD Card Holder
Parts:
- added C13, C14: 100n, SmartPrj:C-EU0603-RND
- added JP1: (no value), pinhead:PINHD-1X1
- added JP2: USD_CONNECTOR, SparkFun-Connectors:USD_CONNECTOR
- added R4, R5, R6, R7: 100k, rcl:R-EU_R0402
- added R_MAX1: 10K, rcl:R-EU_R0402
- added U4: TXB0104, SparkFun-DigitalIC:TXB0104PWRSOIC14
Connections:
- new net !CS_3V3: JP2.!CS, R7.1, U4.A1
- new net CD: JP1.1, JP2.CD2
- new net CDSDSD: JP2.CD1, R6.1
- new net DI_3V3: JP2.DI, U4.A2
- new net DO_3V3: JP2.DO, U4.A4
- new net RSV@1: JP2.RSV@1, R4.1
- new net RSV@2: JP2.RSV@2, R5.1
- new net SCK_3V3: JP2.SCK, U4.A3
- net +3V3: now also C14.2, JP2.VCC, R4.2, R5.2, R7.2, U4.OE, U4.VCCA
- net +5V: now also C13.2, R6.2, U4.VCCB
- net GND: now also C13.1, C14.1, JP2.GND, JP2.SHIELD@1, JP2.SHIELD@3, U4.GND
- net IO9: now also U4.B1
- net MISO: now also U4.B4
- net MOSI: now also U4.B2
- net SCK: now also U4.B3
Other:
- note added: "100KΩ is the max Sandisk recommends"
- note added: "OE must be relative to VCCA"
- note added: "Remove shootthrough current on unused CMOS inputs"
